File: MotorController_Hardware/MotorController_Hardware.sch (KiCad schematic (older format))
At the start: 117 parts, among them Q1 Q_PMOS_DGS, Q2 Q_PMOS_DGS, Q4 FQP30N06L, Q5 FQP30N06L, Q6 FQP30N06L, Q7 FQP30N06L, Q8 FQP30N06L, Q9 FQP30N06L, U1 DRV8301, U2 NUP4201MR6, U3 F28027M, U4 MAX_3232

Commit message: high level layout
Parts:
- removed Conn10: SH_B_M2_PP, MRDT_Connectors:Anderson_1_Horizontal, symbol MotorController_Hardware-rescue:AndersonPP-MRDT_Connectors
- removed Conn11: SH_C_M2_PP, MRDT_Connectors:Anderson_1_Horizontal, symbol MotorController_Hardware-rescue:AndersonPP-MRDT_Connectors
- removed Conn8: AndersonPP, MRDT_Connectors:Anderson_2_Horizontal_Stacked, symbol MotorController_Hardware-rescue:AndersonPP-MRDT_Connectors
- removed Conn9: SH_A_M2_PP, MRDT_Connectors:Anderson_1_Horizontal, symbol MotorController_Hardware-rescue:AndersonPP-MRDT_Connectors
- U3: footprint MRDT_Shields:LAUNCHXL_F28069M_J1_THT_TOP -> MRDT_Shields:F28027M_THT_TOP
Connections:
- net +3V3: now also U3.+3.3V; no longer U3.GND
- net DC_CAL: now also U3.PA3; no longer U3.PD7
- net EN_GATE: now also U3.PA4; no longer U3.PD6
- net GND: now also U3.GND; no longer U3.PF2
- net INH_A: now also U3.PF2
- net INH_B: now also U3.PB3
- net INH_C: now also U3.PC5
- net INL_A: now also U3.PF3
- net INL_B: now also U3.PC4
- net INL_C: now also U3.PC6
- net NFAULT: now also U3.PA6; no longer U3.PA3
- net NOCTW: now also U3.PA7; no longer U3.PA2
- net NSCS: now also U3.PB2; no longer U3.PF3
- net PWM_IN: now also U3.PA2; no longer U3.PF4
- net SCLK: now also U3.PB4; no longer U3.PB6
- net SDI: now also U3.PB7; no longer U3.PC6
- net SDO: now also U3.PB6; no longer U3.PC7
- net UART_RX: now also U3.PB0; no longer U3.PE0
- net UART_TX: now also U3.PB1; no longer U3.PF0
Changed lines of the file:
@@
 Text Notes 14100 10200 0    157  ~ 31
 MAX 3232
-Text GLabel 18700 10450 0    39   Input ~ 0
-PVDD
-$Comp
-L power:GND #PWR050
-U 1 1 5BABDDDC
-P 18700 10650
-F 0 "#PWR050" H 18700 10400 50  0001 C CNN
-F 1 "GND" H 18700 10500 50  0000 C CNN
-F 2 "" H 18700 10650 50  0001 C CNN
-F 3 "" H 18700 10650 50  0001 C CNN
-	1    18700 10650
-	1    0    0    -1
-$EndComp
 Text GLabel 17350 11350 0    39   Input ~ 0
 SH_A
@@
 	1    0    0    -1
 $EndComp
-Text GLabel 18700 11350 0    39   Input ~ 0
-SH_A
-Text GLabel 18700 11750 0    39   Input ~ 0
-SH_B
-Text GLabel 18700 12150 0    39   Input ~ 0
-SH_C
 Wire Wire Line
 	10250 15150 10250 15200
@@
 	17350 12150 17400 12150
 Wire Wire Line
-	18700 11350 18750 11350
-Wire Wire Line
-	18700 11750 18750 11750
-Wire Wire Line
-	18700 12150 18750 12150
-Wire Wire Line
-	18750 10450 18700 10450
-Wire Wire Line
-	18700 10650 18750 10650
-Wire Wire Line
 	17350 10650 17400 10650
 Text GLabel 6300 11750 2    39   Input ~ 0
@@
 Text GLabel 10850 7400 2    39   Input ~ 0
 PVDD
-$Comp
-L MotorController_Hardware-rescue:AndersonPP-MRDT_Connectors Conn9
-U 1 1 5BE3BCAB
-P 19150 11250
-F 0 "Conn9" H 19123 11297 60  0000 R CNN
-F 1 "SH_A_M2_PP" H 19123 11403 60  0000 R CNN
-F 2 "MRDT_Connectors:Anderson_1_Horizontal" H 19000 10700 60  0001 C CNN
-F 3 "" H 19000 10700 60  0001 C CNN
-	1    19150 11250
-	-1   0    0    1
-$EndComp
-$Comp
-L MotorController_Hardware-rescue:AndersonPP-MRDT_Connectors Conn10
-U 1 1 5BE3BE8D
-P 19150 11650
-F 0 "Conn10" H 19123 11697 60  0000 R CNN
-F 1 "SH_B_M2_PP" H 19123 11803 60  0000 R CNN
-F 2 "MRDT_Connectors:Anderson_1_Horizontal" H 19000 11100 60  0001 C CNN
-F 3 "" H 19000 11100 60  0001 C CNN
-	1    19150 11650
-	-1   0    0    1
-$EndComp
-$Comp
-L MotorController_Hardware-rescue:AndersonPP-MRDT_Connectors Conn11
-U 1 1 5BE3C061
-P 19150 12050
-F 0 "Conn11" H 19123 12097 60  0000 R CNN
-F 1 "SH_C_M2_PP" H 19123 12203 60  0000 R CNN
-F 2 "MRDT_Connectors:Anderson_1_Horizontal" H 19000 11500 60  0001 C CNN
-F 3 "" H 19000 11500 60  0001 C CNN
-	1    19150 12050
-	-1   0    0    1
-$EndComp
 $Comp
 L MotorController_Hardware-rescue:AndersonPP-MRDT_Connectors Conn6
@@
 $EndComp
 $Comp
-L MotorController_Hardware-rescue:AndersonPP-MRDT_Connectors Conn8
-U 1 1 5BD6E932
-P 19150 10550
-F 0 "Conn8" H 19123 10597 60  0000 R CNN
-F 1 "AndersonPP" H 19123 10703 60  0000 R CNN
-F 2 "MRDT_Connectors:Anderson_2_Horizontal_Stacked" H 19000 10000 60  0001 C CNN
-F 3 "" H 19000 10000 60  0001 C CNN
-	1    19150 10550
-	-1   0    0    1
-$EndComp
-$Comp
 L MotorController_Hardware-rescue:AndersonPP-MRDT_Connectors Conn3
 U 1 1 5BE3C6D5
@@
 F 3 "" H 17650 10000 60  0001 C CNN
 	1    17800 10550
-	-1   0    0    1
-$EndComp
-$Comp
-L MotorController_Hardware-rescue:AndersonPP-MRDT_Connectors Conn8
-U 4 1 5BF99F47
-P 19150 10350
-F 0 "Conn8" H 19123 10397 60  0000 R CNN
-F 1 "AndersonPP" H 19123 10503 60  0000 R CNN
-F 2 "MRDT_Connectors:Anderson_2_Horizontal_Stacked" H 19000 9800 60  0001 C CNN
-F 3 "" H 19000 9800 60  0001 C CNN
-	4    19150 10350
 	-1   0    0    1
 $EndComp
@@
 Wire Wire Line
 	4500 8150 4500 8350
-$Comp
-L MRDT_Shields:F28027M U3
-U 2 1 5DA7BA5E
-P 14000 8250
-F 0 "U3" H 13800 8150 50  0000 L CNN
-F 1 "F28027M" H 13650 8050 50  0000 L CNN
-F 2 "MRDT_Shields:LAUNCHXL_F28069M_J1_THT_TOP" H 14000 8050 50  0001 C CNN
-F 3 "" H 14000 8050 50  0001 C CNN
-	2    14000 8250
-	1    0    0    -1
-$EndComp
-$Comp
-L MRDT_Shields:F28027M U3
-U 3 1 5DA83779
-P 15500 8250
-F 0 "U3" H 15400 8150 50  0000 C CNN
-F 1 "F28027M" H 15350 8050 50  0000 C CNN
-F 2 "MRDT_Shields:LAUNCHXL_F28069M_J1_THT_TOP" H 15500 8050 50  0001 C CNN
-F 3 "" H 15500 8050 50  0001 C CNN
-	3    15500 8250
-	1    0    0    -1
-$EndComp
 Text GLabel 13600 7600 0    39   Output ~ 0
 UART_TX
@@
 Text GLabel 15100 9250 0    39   Input ~ 0
 SDI
-$Comp
-L MRDT_Shields:F28027M U3
-U 4 1 5DA7F65C
-P 15500 9700
-F 0 "U3" H 15307 10955 50  0000 C CNN
-F 1 "F28027M" H 15350 9600 50  0000 C CNN
-F 2 "MRDT_Shields:LAUNCHXL_F28069M_J1_THT_TOP" H 15500 9500 50  0001 C CNN
-F 3 "" H 15500 9500 50  0001 C CNN
-	4    15500 9700
-	1    0    0    -1
-$EndComp
-$Comp
-L MRDT_Shields:F28027M U3
-U 1 1 5DB93C77
-P 13850 10000
-F 0 "U3" H 13700 10100 50  0000 L CNN
-F 1 "F28027M" H 13600 10200 50  0000 L CNN
-F 2 "MRDT_Shields:LAUNCHXL_F28069M_J1_THT_TOP" H 13850 9800 50  0001 C CNN
-F 3 "" H 13850 9800 50  0001 C CNN
-	1    13850 10000
-	1    0    0    -1
-$EndComp
 Text Notes 12950 9300 0    50   ~ 0
 EPWM3B
@@
 Wire Wire Line
 	16850 13350 16900 13350
+$Comp
+L MRDT_Shields:F28027M U3
+U 1 1 5D9F437D
+P 14000 8250
+F 0 "U3" H 14028 8841 50  0000 L CNN
+F 1 "F28027M" H 14028 8750 50  0000 L CNN
+F 2 "MRDT_Shields:F28027M_THT_TOP" H 14000 8050 50  0001 C CNN
+F 3 "" H 14000 8050 50  0001 C CNN
+	1    14000 8250
+	1    0    0    -1
+$EndComp
+$Comp
+L MRDT_Shields:F28027M U3
+U 2 1 5D9FB202
+P 15500 9700
+F 0 "U3" H 15528 10291 50  0000 L CNN
+F 1 "F28027M" H 15528 10200 50  0000 L CNN
+F 2 "MRDT_Shields:F28027M_THT_TOP" H 15500 9500 50  0001 C CNN
+F 3 "" H 15500 9500 50  0001 C CNN
+	2    15500 9700
+	1    0    0    -1
+$EndComp
+$Comp
+L MRDT_Shields:F28027M U3
+U 3 1 5D9FE18B
+P 15500 8250
+F 0 "U3" H 15528 8841 50  0000 L CNN
+F 1 "F28027M" H 15528 8750 50  0000 L CNN
+F 2 "MRDT_Shields:F28027M_THT_TOP" H 15500 8050 50  0001 C CNN
+F 3 "" H 15500 8050 50  0001 C CNN
+	3    15500 8250
+	1    0    0    -1
+$EndComp
+$Comp
+L MRDT_Shields:F28027M U3
+U 4 1 5DA01419
+P 14000 9700
+F 0 "U3" H 14028 10291 50  0000 L CNN
+F 1 "F28027M" H 14028 10200 50  0000 L CNN
+F 2 "MRDT_Shields:F28027M_THT_TOP" H 14000 9500 50  0001 C CNN
+F 3 "" H 14000 9500 50  0001 C CNN
+	4    14000 9700
+	1    0    0    -1
+$EndComp
 $EndSCHEMATC

Commit message: Work done on PCB layout
Parts:
- C36: value C_Small -> .015 uF
- U3: symbol MRDT_Shields:F28027M -> MotorController_Hardware-rescue:F28027M-MRDT_Shields
Connections:
- net VCC is gone; now on net +3V3: D2.2 (A), Q1.3 (S), Q2.3 (S)
- net +3V3: now also U2.5 (VP); no longer U2.2 (VN)
- net GND: now also U2.2 (VN); no longer U2.5 (VP)
- net PWM_IN: now also C36.1, R7.2
Other:
- note added: "WAS\nVN = 3.3V\nVP = GND"
- note added: "Was 3.3V, why?"

Commit message: Finished PCB layout
Parts:
- +3V3: footprint Package_TO_SOT_SMD:SOT-23_Handsoldering -> MRDT_Drill_Holes:Via_.6mm
Connections:
- net at C13.1, D1.1 (K), L1.2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: now also U1.51 (PH)
Other:
- note removed: "Was 3.3V, why?"
Changed lines of the file:
@@
 Wire Wire Line
 	6400 7650 7600 7650
-Connection ~ 6400 8250
 Wire Wire Line
 	6400 8250 6700 8250
@@
 F 3 "" H 6050 13050 394 0001 C CNN
 	3    5450 11100
-	1    0    0    -1
-$EndComp
-$Comp
-L MotorController_Hardware-rescue:DRV8301-MRDT_ICs U1
-U 4 1 5BC930B8
-P 5200 8450
-F 0 "U1" H 5300 8400 59  0000 C CNN
-F 1 "DRV8301" H 5450 8400 69  0001 C CNN
-F 2 "MRDT_ICs:DRV8301" H 5800 10400 394 0001 C CNN
-F 3 "" H 5800 10400 394 0001 C CNN
-	4    5200 8450
 	1    0    0    -1
 $EndComp
@@
 F 0 "+3V3" H 4150 11050 50  0000 C BNN
 F 1 "TEST" H 4150 11000 50  0000 C CNN
-F 2 "Package_TO_SOT_SMD:SOT-23_Handsoldering" H 4150 10750 50  0001 C CNN
+F 2 "MRDT_Drill_Holes:Via_.6mm" H 4150 10750 50  0001 C CNN
 F 3 "" H 4150 10750 50  0001 C CNN
 	1    4150 10750
@@
 Wire Wire Line
 	6650 9050 6950 9050
-Wire Wire Line
-	6150 9050 6650 9050
 Connection ~ 6650 9050
-Wire Wire Line
-	6150 8850 6650 8850
 Wire Wire Line
 	6400 8050 6700 8050
@@
 Connection ~ 4500 8150
 Wire Wire Line
-	4500 8350 5000 8350
+	4500 8350 4850 8350
 Wire Wire Line
 	4450 8350 4500 8350
@@
 Wire Wire Line
 	4350 10650 4350 10750
-Text Notes 4400 10450 0    50   ~ 0
-Was 3.3V, why?
-Text Notes 3900 7950 0    50   ~ 0
-Was 3.3V, why?
 Text Notes 6250 14950 0    50   ~ 0
 WAS\nVN = 3.3V\nVP = GND
 $Comp
-L power:+3.3V #PWR?
+L power:+3.3V #PWR0112
 U 1 1 5DA34D1C
 P 6750 14950
-F 0 "#PWR?" H 6750 14800 50  0001 C CNN
+F 0 "#PWR0112" H 6750 14800 50  0001 C CNN
 F 1 "+3.3V" H 6765 15123 50  0000 C CNN
 F 2 "" H 6750 14950 50  0001 C CNN
@@
 $EndComp
 $Comp
-L power:+3.3V #PWR?
+L power:+3.3V #PWR0113
 U 1 1 5DA354EC
 P 4350 10650
-F 0 "#PWR?" H 4350 10500 50  0001 C CNN
+F 0 "#PWR0113" H 4350 10500 50  0001 C CNN
 F 1 "+3.3V" H 4365 10823 50  0000 C CNN
 F 2 "" H 4350 10650 50  0001 C CNN
@@
 $EndComp
 $Comp
-L power:+3.3V #PWR?
+L power:+3.3V #PWR0114
 U 1 1 5DA367CF
 P 3800 8050
-F 0 "#PWR?" H 3800 7900 50  0001 C CNN
+F 0 "#PWR0114" H 3800 7900 50  0001 C CNN
 F 1 "+3.3V" H 3815 8223 50  0000 C CNN
 F 2 "" H 3800 8050 50  0001 C CNN
@@
 $EndComp
 $Comp
-L power:+3.3V #PWR?
+L power:+3.3V #PWR0115
 U 1 1 5DA391C2
 P 14600 13350
-F 0 "#PWR?" H 14600 13200 50  0001 C CNN
+F 0 "#PWR0115" H 14600 13200 50  0001 C CNN
 F 1 "+3.3V" H 14615 13523 50  0000 C CNN
 F 2 "" H 14600 13350 50  0001 C CNN
@@
 $EndComp
 $Comp
-L power:+3.3V #PWR?
+L power:+3.3V #PWR0117
 U 1 1 5DA3A512
 P 16150 13050
-F 0 "#PWR?" H 16150 12900 50  0001 C CNN
+F 0 "#PWR0117" H 16150 12900 50  0001 C CNN
 F 1 "+3.3V" H 16300 13150 50  0000 C CNN
 F 2 "" H 16150 13050 50  0001 C CNN
@@
 	1    0    0    -1
 $EndComp
+Connection ~ 6400 8250
+Wire Wire Line
+	6150 8850 6650 8850
+Wire Wire Line
+	6150 9050 6650 9050
+$Comp
+L MotorController_Hardware-rescue:DRV8301-MRDT_ICs U1
+U 4 1 5BC930B8
+P 5200 8450
+F 0 "U1" H 5300 8400 59  0000 C CNN
+F 1 "DRV8301" H 5450 8400 69  0001 C CNN
+F 2 "MRDT_ICs:DRV8301" H 5800 10400 394 0001 C CNN
+F 3 "" H 5800 10400 394 0001 C CNN
+	4    5200 8450
+	1    0    0    -1
+$EndComp
+Wire Wire Line
+	5000 8250 4850 8250
+Wire Wire Line
+	4850 8250 4850 8350
+Connection ~ 4850 8350
+Wire Wire Line
+	4850 8350 5000 8350
 $EndSCHEMATC

Commit message: Silkscreens added
Parts:
- GHA_M1, GHB_M1, GHC_M1, GLA_M1, GLB_M1, GLC_M1, PVDD_M1, SHA_M1, SHB_M1, SHC_M1: footprint Wire_Pads:SolderWirePad_single_1mmDrill -> MRDT_Drill_Holes:Via_.6mm
Changed lines of the file:
@@
 F 0 "SHA_M1" H 11650 8500 50  0000 C BNN
 F 1 "TEST" H 11650 8450 50  0000 C CNN
-F 2 "Wire_Pads:SolderWirePad_single_1mmDrill" H 11650 8200 50  0001 C CNN
+F 2 "MRDT_Drill_Holes:Via_.6mm" H 11650 8200 50  0001 C CNN
 F 3 "" H 11650 8200 50  0001 C CNN
 	1    11650 8200
@@
 F 0 "GLA_M1" H 10250 8900 50  0000 C BNN
 F 1 "TEST" H 10250 8850 50  0000 C CNN
-F 2 "Wire_Pads:SolderWirePad_single_1mmDrill" H 10250 8600 50  0001 C CNN
+F 2 "MRDT_Drill_Holes:Via_.6mm" H 10250 8600 50  0001 C CNN
 F 3 "" H 10250 8600 50  0001 C CNN
 	1    10250 8600
@@
 F 0 "GHB_M1" H 10250 11150 50  0000 C BNN
 F 1 "TEST" H 10250 11100 50  0000 C CNN
-F 2 "Wire_Pads:SolderWirePad_single_1mmDrill" H 10250 10850 50  0001 C CNN
+F 2 "MRDT_Drill_Holes:Via_.6mm" H 10250 10850 50  0001 C CNN
 F 3 "" H 10250 10850 50  0001 C CNN
 	1    10250 10850
@@
 F 0 "SHB_M1" H 11650 11650 50  0000 C BNN
 F 1 "TEST" H 11650 11600 50  0000 C CNN
-F 2 "Wire_Pads:SolderWirePad_single_1mmDrill" H 11650 11350 50  0001 C CNN
+F 2 "MRDT_Drill_Holes:Via_.6mm" H 11650 11350 50  0001 C CNN
 F 3 "" H 11650 11350 50  0001 C CNN
 	1    11650 11350
@@
 F 0 "GLB_M1" H 10250 12050 50  0000 C BNN
 F 1 "TEST" H 10250 12000 50  0000 C CNN
-F 2 "Wire_Pads:SolderWirePad_single_1mmDrill" H 10250 11750 50  0001 C CNN
+F 2 "MRDT_Drill_Holes:Via_.6mm" H 10250 11750 50  0001 C CNN
 F 3 "" H 10250 11750 50  0001 C CNN
 	1    10250 11750
@@
 F 0 "GHC_M1" H 10250 14500 50  0000 C BNN
 F 1 "TEST" H 10250 14450 50  0000 C CNN
-F 2 "Wire_Pads:SolderWirePad_single_1mmDrill" H 10250 14200 50  0001 C CNN
+F 2 "MRDT_Drill_Holes:Via_.6mm" H 10250 14200 50  0001 C CNN
 F 3 "" H 10250 14200 50  0001 C CNN
 	1    10250 14200
@@
 F 0 "SHC_M1" H 11650 15000 50  0000 C BNN
 F 1 "TEST" H 11650 14950 50  0000 C CNN
-F 2 "Wire_Pads:SolderWirePad_single_1mmDrill" H 11650 14700 50  0001 C CNN
+F 2 "MRDT_Drill_Holes:Via_.6mm" H 11650 14700 50  0001 C CNN
 F 3 "" H 11650 14700 50  0001 C CNN
 	1    11650 14700
@@
 F 0 "GLC_M1" H 10250 15400 50  0000 C BNN
 F 1 "TEST" H 10250 15350 50  0000 C CNN
-F 2 "Wire_Pads:SolderWirePad_single_1mmDrill" H 10250 15100 50  0001 C CNN
+F 2 "MRDT_Drill_Holes:Via_.6mm" H 10250 15100 50  0001 C CNN
 F 3 "" H 10250 15100 50  0001 C CNN
 	1    10250 15100
@@
 F 0 "PVDD_M1" H 3600 14650 50  0000 L CNN
 F 1 "TEST" H 3600 14550 50  0000 L CNN
-F 2 "Wire_Pads:SolderWirePad_single_1mmDrill" H 3900 14350 50  0001 C CNN
+F 2 "MRDT_Drill_Holes:Via_.6mm" H 3900 14350 50  0001 C CNN
 F 3 "~" H 3900 14350 50  0001 C CNN
 	1    3700 14350
@@
 F 0 "GHA_M1" H 10250 8000 50  0000 C BNN
 F 1 "tp" H 10250 7950 50  0000 C CNN
-F 2 "Wire_Pads:SolderWirePad_single_1mmDrill" H 10250 7700 50  0001 C CNN
+F 2 "MRDT_Drill_Holes:Via_.6mm" H 10250 7700 50  0001 C CNN
 F 3 "" H 10250 7700 50  0001 C CNN
 	1    10250 7700

Commit message: WORKING ON ORDERING
Parts:
- removed D1: D_Shottky, Diode_SMD:D_SOD-123, symbol Device:D_Schottky
- added D1: D_Zener, Diode_SMD:D_0603_1608Metric_Pad1.05x0.95mm_HandSolder, symbol Device:D_Zener
- added D5: LED, Inductor_SMD:L_0603_1608Metric_Pad1.05x0.95mm_HandSolder, symbol Device:LED
- added R17, R21: 0, Resistor_SMD:R_0603_1608Metric_Pad1.05x0.95mm_HandSolder, symbol Device:R
- added R36: 1000, Resistor_SMD:R_0603_1608Metric_Pad1.05x0.95mm_HandSolder, symbol Device:R
- R7: value R -> 100
- R9: value 500 -> 510
Connections:
- net GND: now also D1.2 (A), R17.1, R21.1, R36.2; no longer U1.30 (SP2), U1.32 (SP1)
- net PVDD: now also D5.2 (A)
- net at C13.1, L1.2, U1.50 (PH)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: now also D1.1 (K)
- new net: D5.1 (K), R36.1
- new net SP1: R17.2, U1.32 (SP1)
- new net SP2: R21.2, U1.30 (SP2)
Changed lines of the file:
@@
 L power:GND #PWR019
 U 1 1 5BA8117C
-P 6150 11050
-F 0 "#PWR019" H 6150 10800 50  0001 C CNN
-F 1 "GND" H 6150 10900 50  0000 C CNN
-F 2 "" H 6150 11050 50  0001 C CNN
-F 3 "" H 6150 11050 50  0001 C CNN
-	1    6150 11050
+P 6200 11050
+F 0 "#PWR019" H 6200 10800 50  0001 C CNN
+F 1 "GND" H 6200 10900 50  0000 C CNN
+F 2 "" H 6200 11050 50  0001 C CNN
+F 3 "" H 6200 11050 50  0001 C CNN
+	1    6200 11050
 	1    0    0    -1
 $EndComp
@@
 Connection ~ 6300 12550
 Wire Wire Line
-	6250 12050 6800 12050
-Wire Wire Line
-	6800 11850 6800 12050
-Connection ~ 6800 12050
-Wire Wire Line
-	6250 11850 6800 11850
-Wire Wire Line
 	6650 12450 6800 12450
 Wire Wire Line
 	6800 12450 6800 12500
-Wire Wire Line
-	6800 12050 6800 12450
-Connection ~ 6800 12450
 Wire Wire Line
 	5100 12650 5150 12650
@@
 	1    3500 8300
 	1    0    0    -1
-$EndComp
-$Comp
-L Device:D_Schottky D1
-U 1 1 5BA6C283
-P 4300 8350
-F 0 "D1" H 4300 8450 50  0000 C CNN
-F 1 "D_Shottky" H 4300 8250 50  0000 C CNN
-F 2 "Diode_SMD:D_SOD-123" H 4300 8350 50  0001 C CNN
-F 3 "" H 4300 8350 50  0001 C CNN
-	1    4300 8350
-	-1   0    0    1
 $EndComp
 $Comp
@@
 P 14600 12250
 F 0 "R7" V 14700 12250 50  0000 C CNN
-F 1 "R" V 14600 12250 50  0000 C CNN
+F 1 "100" V 14600 12250 50  0000 C CNN
 F 2 "Resistor_SMD:R_0603_1608Metric_Pad1.05x0.95mm_HandSolder" V 14530 12250 50  0001 C CNN
 F 3 "~" H 14600 12250 50  0001 C CNN
@@
 P 14600 13900
 F 0 "R9" H 14670 13946 50  0000 L CNN
-F 1 "500" H 14670 13855 50  0000 L CNN
+F 1 "510" V 14600 13800 50  0000 L CNN
 F 2 "Resistor_SMD:R_0603_1608Metric_Pad1.05x0.95mm_HandSolder" V 14530 13900 50  0001 C CNN
 F 3 "~" H 14600 13900 50  0001 C CNN
@@
 Wire Wire Line
 	4850 8350 5000 8350
+$Comp
+L Device:D_Zener D1
+U 1 1 5DABAAD8
+P 4300 8350
+F 0 "D1" H 4300 8250 50  0000 C CNN
+F 1 "D_Zener" H 4300 8500 50  0000 C CNN
+F 2 "Diode_SMD:D_0603_1608Metric_Pad1.05x0.95mm_HandSolder" H 4300 8350 50  0001 C CNN
+F 3 "~" H 4300 8350 50  0001 C CNN
+	1    4300 8350
+	-1   0    0    1
+$EndComp
+Connection ~ 10450 9500
+Wire Wire Line
+	6150 11050 6200 11050
+Text GLabel 6300 11850 2    39   Input ~ 0
+SP1
+Wire Wire Line
+	6250 11850 6300 11850
+Text GLabel 9400 9500 0    39   Input ~ 0
+SP1
+$Comp
+L Device:R R17
+U 1 1 5DDD2663
+P 9850 9500
+F 0 "R17" V 9750 9500 50  0000 C CNN
+F 1 "0" V 9850 9500 50  0000 C CNN
+F 2 "Resistor_SMD:R_0603_1608Metric_Pad1.05x0.95mm_HandSolder" V 9780 9500 50  0001 C CNN
+F 3 "~" H 9850 9500 50  0001 C CNN
+	1    9850 9500
+	0    1    1    0
+$EndComp
+Text GLabel 6300 12050 2    39   Input ~ 0
+SP2
+Wire Wire Line
+	6300 12050 6250 12050
+Text GLabel 9950 12650 0    39   Input ~ 0
+SP2
+Wire Wire Line
+	10350 12650 10450 12650
+Connection ~ 10450 12650
+$Comp
+L Device:R R21
+U 1 1 5DEBA21A
+P 10200 12650
+F 0 "R21" V 10100 12650 50  0000 C CNN
+F 1 "0" V 10200 12650 50  0000 C CNN
+F 2 "Resistor_SMD:R_0603_1608Metric_Pad1.05x0.95mm_HandSolder" V 10130 12650 50  0001 C CNN
+F 3 "~" H 10200 12650 50  0001 C CNN
+	1    10200 12650
+	0    1    1    0
+$EndComp
+Wire Wire Line
+	9950 12650 10050 12650
+$Comp
+L Device:R R36
+U 1 1 5DF4C982
+P 14000 13900
+F 0 "R36" H 14070 13946 50  0000 L CNN
+F 1 "1000" V 14000 13800 50  0000 L CNN
+F 2 "Resistor_SMD:R_0603_1608Metric_Pad1.05x0.95mm_HandSolder" V 13930 13900 50  0001 C CNN
+F 3 "~" H 14000 13900 50  0001 C CNN
+	1    14000 13900
+	1    0    0    -1
+$EndComp
+$Comp
+L Device:LED D5
+U 1 1 5DF4C988
+P 14000 13550
+F 0 "D5" V 14039 13433 50  0000 R CNN
+F 1 "LED" V 13948 13433 50  0000 R CNN
+F 2 "Inductor_SMD:L_0603_1608Metric_Pad1.05x0.95mm_HandSolder" H 14000 13550 50  0001 C CNN
+F 3 "~" H 14000 13550 50  0001 C CNN
+	1    14000 13550
+	0    -1   -1   0
+$EndComp
+Wire Wire Line
+	14000 13700 14000 13750
+Wire Wire Line
+	14000 13400 14000 13350
+$Comp
+L power:GND #PWR0119
+U 1 1 5DF4C990
+P 14000 14200
+F 0 "#PWR0119" H 14000 13950 50  0001 C CNN
+F 1 "GND" H 14005 14027 50  0000 C CNN
+F 2 "" H 14000 14200 50  0001 C CNN
+F 3 "" H 14000 14200 50  0001 C CNN
+	1    14000 14200
+	1    0    0    -1
+$EndComp
+Wire Wire Line
+	14000 14050 14000 14200
+Text GLabel 14000 13350 1    39   Input ~ 0
+PVDD
+Wire Wire Line
+	9400 9500 9700 9500
+Wire Wire Line
+	10000 9500 10450 9500
 $EndSCHEMATC
