File: MotorController_Hardware/MotorController_Hardware.kicad_pcb (KiCad board)
At the start: 4 copper layers, 112.9 x 80 mm, 117 parts, among them Q1 Q_PMOS_DGS, Q2 Q_PMOS_DGS, Q4 FQP30N06L, Q5 FQP30N06L, Q6 FQP30N06L, Q7 FQP30N06L, Q8 FQP30N06L, Q9 FQP30N06L, U1 DRV8301, U2 NUP4201MR6, U3 F28027M, U4 MAX_3232

Commit message: BOM update
Parts:
- added REF**: 6_32_Hole, MRDT_Drill_Holes:6_32_Hole_Corner, F.Cu at (93.4, 64.1)
- added REF**: 6_32_Hole, MRDT_Drill_Holes:6_32_Hole_Corner, F.Cu at (93.5, 125.5)
- added REF**: 6_32_Hole, MRDT_Drill_Holes:6_32_Hole_Corner, F.Cu at (187.8, 125.6)
- added REF**: 6_32_Hole, MRDT_Drill_Holes:6_32_Hole_Corner, F.Cu at (211.6, 113.2)
- added REF**: 6_32_Hole, MRDT_Drill_Holes:6_32_Hole_Corner, F.Cu at (187.6, 64.1)
- moved C5 0.39 mm to (98.0, 63.7)
Changed lines of the file:
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@@
     (tracks 963)
     (zones 0)
-    (modules 117)
+    (modules 122)
     (nets 101)
   )
@@
   )
   (setup
-    (last_trace_width 0.381)
+    (last_trace_width 0.25)
     (user_trace_width 0.254)
     (user_trace_width 0.3048)
@@
     (add_net UART_RX)
     (add_net UART_TX)
+  )
+  (module MRDT_Drill_Holes:6_32_Hole_Corner (layer F.Cu)
+    (at 93.4085 64.0715 90)
+    (fp_text reference REF** (at 4.445 -3.945 90) (layer F.SilkS) hide
+      (effects (font (size 1 1) (thickness 0.15)))
+    )
+    (fp_text value 6_32_Hole (at 4.445 -4.945 90) (layer F.Fab)
+      (effects (font (size 1 1) (thickness 0.15)))
+    )
+    (fp_line (start 8.89 0) (end 8.89 -4.445) (layer F.Fab) (width 0.15))
+    (fp_line (start 4.445 0) (end 8.89 0) (layer F.Fab) (width 0.15))
+    (fp_line (start 0 -8.89) (end 4.445 -8.89) (layer F.Fab) (width 0.15))
+    (fp_line (start 0 -4.445) (end 0 -8.89) (layer F.Fab) (width 0.15))
+    (fp_line (start 0 0) (end 0 -4.445) (layer F.Fab) (width 0.15))
+    (fp_line (start 4.445 0) (end 0 0) (layer F.Fab) (width 0.15))
+    (fp_circle (center 4.445 -4.445) (end 8.89 -4.445) (layer F.SilkS) (width 0.15))
+    (pad "" np_thru_hole circle (at 4.445 -4.445 90) (size 3.683 3.683) (drill 3.683) (layers *.Cu *.Mask))
+  )
+  (module MRDT_Drill_Holes:6_32_Hole_Corner (layer F.Cu)
+    (at 93.472 125.5395 180)
+    (fp_text reference REF** (at 4.445 -3.945) (layer F.SilkS) hide
+      (effects (font (size 1 1) (thickness 0.15)))
+    )
+    (fp_text value 6_32_Hole (at 4.445 -4.945) (layer F.Fab)
+      (effects (font (size 1 1) (thickness 0.15)))
+    )
+    (fp_line (start 8.89 0) (end 8.89 -4.445) (layer F.Fab) (width 0.15))
+    (fp_line (start 4.445 0) (end 8.89 0) (layer F.Fab) (width 0.15))
+    (fp_line (start 0 -8.89) (end 4.445 -8.89) (layer F.Fab) (width 0.15))
+    (fp_line (start 0 -4.445) (end 0 -8.89) (layer F.Fab) (width 0.15))
+    (fp_line (start 0 0) (end 0 -4.445) (layer F.Fab) (width 0.15))
+    (fp_line (start 4.445 0) (end 0 0) (layer F.Fab) (width 0.15))
+    (fp_circle (center 4.445 -4.445) (end 8.89 -4.445) (layer F.SilkS) (width 0.15))
+    (pad "" np_thru_hole circle (at 4.445 -4.445 180) (size 3.683 3.683) (drill 3.683) (layers *.Cu *.Mask))
+  )
+  (module MRDT_Drill_Holes:6_32_Hole_Corner (layer F.Cu)
+    (at 187.833 125.603 270)
+    (fp_text reference REF** (at 4.445 -3.945 90) (layer F.SilkS) hide
+      (effects (font (size 1 1) (thickness 0.15)))
+    )
+    (fp_text value 6_32_Hole (at 4.445 -4.945 90) (layer F.Fab)
+      (effects (font (size 1 1) (thickness 0.15)))
+    )
+    (fp_line (start 8.89 0) (end 8.89 -4.445) (layer F.Fab) (width 0.15))
+    (fp_line (start 4.445 0) (end 8.89 0) (layer F.Fab) (width 0.15))
+    (fp_line (start 0 -8.89) (end 4.445 -8.89) (layer F.Fab) (width 0.15))
+    (fp_line (start 0 -4.445) (end 0 -8.89) (layer F.Fab) (width 0.15))
+    (fp_line (start 0 0) (end 0 -4.445) (layer F.Fab) (width 0.15))
+    (fp_line (start 4.445 0) (end 0 0) (layer F.Fab) (width 0.15))
+    (fp_circle (center 4.445 -4.445) (end 8.89 -4.445) (layer F.SilkS) (width 0.15))
+    (pad "" np_thru_hole circle (at 4.445 -4.445 270) (size 3.683 3.683) (drill 3.683) (layers *.Cu *.Mask))
+  )
+  (module MRDT_Drill_Holes:6_32_Hole_Corner (layer F.Cu)
+    (at 211.6455 113.2205)
+    (fp_text reference REF** (at 4.445 -3.945) (layer F.SilkS) hide
+      (effects (font (size 1 1) (thickness 0.15)))
+    )
+    (fp_text value 6_32_Hole (at 4.445 -4.945) (layer F.Fab)
+      (effects (font (size 1 1) (thickness 0.15)))
+    )
+    (fp_circle (center 4.445 -4.445) (end 8.89 -4.445) (layer F.SilkS) (width 0.15))
+    (fp_line (start 4.445 0) (end 0 0) (layer F.Fab) (width 0.15))
+    (fp_line (start 0 0) (end 0 -4.445) (layer F.Fab) (width 0.15))
+    (fp_line (start 0 -4.445) (end 0 -8.89) (layer F.Fab) (width 0.15))
+    (fp_line (start 0 -8.89) (end 4.445 -8.89) (layer F.Fab) (width 0.15))
+    (fp_line (start 4.445 0) (end 8.89 0) (layer F.Fab) (width 0.15))
+    (fp_line (start 8.89 0) (end 8.89 -4.445) (layer F.Fab) (width 0.15))
+    (pad "" np_thru_hole circle (at 4.445 -4.445) (size 3.683 3.683) (drill 3.683) (layers *.Cu *.Mask))
+  )
+  (module MRDT_Drill_Holes:6_32_Hole_Corner (layer F.Cu)
+    (at 187.6425 64.0715)
+    (fp_text reference REF** (at 4.445 -3.945) (layer F.SilkS) hide
+      (effects (font (size 1 1) (thickness 0.15)))
+    )
+    (fp_text value 6_32_Hole (at 4.445 -4.945) (layer F.Fab)
+      (effects (font (size 1 1) (thickness 0.15)))
+    )
+    (fp_line (start 8.89 0) (end 8.89 -4.445) (layer F.Fab) (width 0.15))
+    (fp_line (start 4.445 0) (end 8.89 0) (layer F.Fab) (width 0.15))
+    (fp_line (start 0 -8.89) (end 4.445 -8.89) (layer F.Fab) (width 0.15))
+    (fp_line (start 0 -4.445) (end 0 -8.89) (layer F.Fab) (width 0.15))
+    (fp_line (start 0 0) (end 0 -4.445) (layer F.Fab) (width 0.15))
+    (fp_line (start 4.445 0) (end 0 0) (layer F.Fab) (width 0.15))
+    (fp_circle (center 4.445 -4.445) (end 8.89 -4.445) (layer F.SilkS) (width 0.15))
+    (pad "" np_thru_hole circle (at 4.445 -4.445) (size 3.683 3.683) (drill 3.683) (layers *.Cu *.Mask))
   )
   (module MRDT_ICs:DRV8301 (layer F.Cu)
@@
   )
   (module Capacitor_THT:CP_Radial_D12.5mm_P5.00mm (layer F.Cu)
-    (at 97.663 63.754 90)
+    (at 98.044 63.6905 90)
     (descr "CP, Radial series, Radial, pin pitch=5.00mm, , diameter=12.5mm, Electrolytic Capacitor")
     (tags "CP Radial series Radial pin pitch 5.00mm  diameter 12.5mm Electrolytic Capacitor")
